File: VFD_Watch.sch (KiCad schematic (older format))
At the start: 52 parts, among them J1 USB_B_Micro, J2 I2C_Con, Q1 MBT3904DW1, SW1 B1, SW2 B2, SW3 B_RES, SW4 B_0, U1 MIC5219-3.3YM5, U2 DRV8837C, U3 MP3120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

Commit message: fixed BAT INPUT to allow for LiPo voltages without damaging the ESP32, cleaned up silkscreen, updated graphics
Parts:
- added R18, R19: 10k, Resistor_SMD:R_0805_2012Metric, symbol Device:R
- U4: symbol Interface_USB:FT231XS -> VFD_Watch-rescue:FT231XS-Interface_USB
Connections:
- net +BATT: now also R18.1; no longer U6.6 (IO34)
- net GND: now also R19.2
- new net: R18.2, R19.1, U6.6 (IO34)
Other:
- moved on the sheet: C18, R16, SW3
Changed lines of the file:
@@
 EESchema Schematic File Version 4
 LIBS:VFD_Watch-cache
-EELAYER 28 0
+EELAYER 29 0
 EELAYER END
 $Descr A4 11693 8268
@@
 Title ""
 Date ""
-Rev ""
+Rev "1.1"
 Comp ""
 Comment1 ""
@@
 $EndComp
 $Comp
-L Interface_USB:FT231XS U4
+L VFD_Watch-rescue:FT231XS-Interface_USB U4
 U 1 1 5BE511C0
 P 3500 1850
@@
 L Device:R R16
 U 1 1 5C093024
-P 7200 1650
-F 0 "R16" H 7270 1696 50  0000 L CNN
-F 1 "10k" H 7270 1605 50  0000 L CNN
-F 2 "Resistor_SMD:R_0805_2012Metric" V 7130 1650 50  0001 C CNN
-F 3 "~" H 7200 1650 50  0001 C CNN
-	1    7200 1650
-	1    0    0    -1
-$EndComp
-Wire Wire Line
-	7200 1500 7200 1450
-Wire Wire Line
-	7200 1450 7750 1450
+P 7150 1650
+F 0 "R16" H 7220 1696 50  0000 L CNN
+F 1 "10k" H 7220 1605 50  0000 L CNN
+F 2 "Resistor_SMD:R_0805_2012Metric" V 7080 1650 50  0001 C CNN
+F 3 "~" H 7150 1650 50  0001 C CNN
+	1    7150 1650
+	1    0    0    -1
+$EndComp
+Wire Wire Line
+	7150 1500 7150 1450
+Wire Wire Line
+	7150 1450 7750 1450
 Connection ~ 7750 1450
 Wire Wire Line
 	7750 1450 7750 1750
 Wire Wire Line
-	7200 1800 7200 1850
-Wire Wire Line
-	7200 1850 7950 1850
+	7150 1800 7150 1850
+Wire Wire Line
+	7150 1850 7950 1850
 $Comp
 L power:GND #PWR0116
 U 1 1 5C0A5AEB
-P 7200 2350
-F 0 "#PWR0116" H 7200 2100 50  0001 C CNN
-F 1 "GND" H 7205 2177 50  0000 C CNN
-F 2 "" H 7200 2350 50  0001 C CNN
-F 3 "" H 7200 2350 50  0001 C CNN
-	1    7200 2350
+P 7150 2350
+F 0 "#PWR0116" H 7150 2100 50  0001 C CNN
+F 1 "GND" H 7155 2177 50  0000 C CNN
+F 2 "" H 7150 2350 50  0001 C CNN
+F 3 "" H 7150 2350 50  0001 C CNN
+	1    7150 2350
 	1    0    0    -1
 $EndComp
@@
 L Switch:SW_Push SW3
 U 1 1 5C0A6DC7
-P 7200 2100
-F 0 "SW3" V 7246 2052 50  0000 R CNN
-F 1 "B_RES" V 7155 2052 50  0000 R CNN
-F 2 "Button_Switch_SMD:SW_SPST_EVQP7A" H 7200 2300 50  0001 C CNN
-F 3 "" H 7200 2300 50  0001 C CNN
-	1    7200 2100
+P 7150 2100
+F 0 "SW3" V 7196 2052 50  0000 R CNN
+F 1 "B_RES" V 7105 2052 50  0000 R CNN
+F 2 "Button_Switch_SMD:SW_SPST_EVQP7A" H 7150 2300 50  0001 C CNN
+F 3 "" H 7150 2300 50  0001 C CNN
+	1    7150 2100
 	0    -1   -1   0
 $EndComp
 Wire Wire Line
-	7200 1900 7200 1850
-Connection ~ 7200 1850
-Wire Wire Line
-	7200 2300 7200 2350
-Text GLabel 6800 1850 0    50   Input ~ 0
+	7150 1900 7150 1850
+Connection ~ 7150 1850
+Wire Wire Line
+	7150 2300 7150 2350
+Text GLabel 6750 1850 0    50   Input ~ 0
 ENABLE
 Wire Wire Line
-	6800 1850 6850 1850
+	6750 1850 6800 1850
 Text GLabel 5100 1100 1    50   Input ~ 0
 ENABLE
@@
 L Device:C C18
 U 1 1 5C1880C2
-P 6850 2150
-F 0 "C18" H 6850 2350 50  0000 L CNN
-F 1 "100nF" H 6850 2250 50  0000 L CNN
-F 2 "Capacitor_SMD:C_0805_2012Metric" H 6888 2000 50  0001 C CNN
-F 3 "~" H 6850 2150 50  0001 C CNN
-	1    6850 2150
-	1    0    0    -1
-$EndComp
-Wire Wire Line
-	6850 2000 6850 1850
-Connection ~ 6850 1850
-Wire Wire Line
-	6850 1850 7200 1850
+P 6800 2150
+F 0 "C18" H 6800 2350 50  0000 L CNN
+F 1 "100nF" H 6800 2250 50  0000 L CNN
+F 2 "Capacitor_SMD:C_0805_2012Metric" H 6838 2000 50  0001 C CNN
+F 3 "~" H 6800 2150 50  0001 C CNN
+	1    6800 2150
+	1    0    0    -1
+$EndComp
+Wire Wire Line
+	6800 2000 6800 1850
+Connection ~ 6800 1850
+Wire Wire Line
+	6800 1850 7150 1850
 $Comp
 L power:GND #PWR0119
 U 1 1 5C19D741
-P 6850 2350
-F 0 "#PWR0119" H 6850 2100 50  0001 C CNN
-F 1 "GND" H 6855 2177 50  0000 C CNN
-F 2 "" H 6850 2350 50  0001 C CNN
-F 3 "" H 6850 2350 50  0001 C CNN
-	1    6850 2350
-	1    0    0    -1
-$EndComp
-Wire Wire Line
-	6850 2350 6850 2300
+P 6800 2350
+F 0 "#PWR0119" H 6800 2100 50  0001 C CNN
+F 1 "GND" H 6805 2177 50  0000 C CNN
+F 2 "" H 6800 2350 50  0001 C CNN
+F 3 "" H 6800 2350 50  0001 C CNN
+	1    6800 2350
+	1    0    0    -1
+$EndComp
+Wire Wire Line
+	6800 2350 6800 2300
 $Comp
 L Device:R R17
@@
 L power:+BATT #PWR0128
 U 1 1 5C4DB255
-P 7750 2100
-F 0 "#PWR0128" H 7750 1950 50  0001 C CNN
-F 1 "+BATT" H 7765 2273 50  0000 C CNN
-F 2 "" H 7750 2100 50  0001 C CNN
-F 3 "" H 7750 2100 50  0001 C CNN
-	1    7750 2100
-	1    0    0    -1
-$EndComp
-Wire Wire Line
-	7750 2100 7750 2150
+P 7500 2100
+F 0 "#PWR0128" H 7500 1950 50  0001 C CNN
+F 1 "+BATT" H 7515 2273 50  0000 C CNN
+F 2 "" H 7500 2100 50  0001 C CNN
+F 3 "" H 7500 2100 50  0001 C CNN
+	1    7500 2100
+	1    0    0    -1
+$EndComp
 Wire Wire Line
 	7750 2150 7950 2150
@@
 	7750 800  7750 1450
 $Comp
-L power:GND #PWR?
+L power:GND #PWR0142
 U 1 1 5BF4566A
 P 7200 1200
-F 0 "#PWR?" H 7200 950 50  0001 C CNN
+F 0 "#PWR0142" H 7200 950 50  0001 C CNN
 F 1 "GND" H 7205 1027 50  0000 C CNN
 F 2 "" H 7200 1200 50  0001 C CNN
@@
 Wire Wire Line
 	2350 1550 2800 1550
+$Comp
+L Device:R R18
+U 1 1 5DC82C16
+P 7500 2300
+F 0 "R18" H 7570 2346 50  0000 L CNN
+F 1 "10k" H 7570 2255 50  0000 L CNN
+F 2 "Resistor_SMD:R_0805_2012Metric" V 7430 2300 50  0001 C CNN
+F 3 "~" H 7500 2300 50  0001 C CNN
+	1    7500 2300
+	1    0    0    -1
+$EndComp
+Wire Wire Line
+	7500 2100 7500 2150
+$Comp
+L Device:R R19
+U 1 1 5DCCA3D6
+P 7500 2700
+F 0 "R19" H 7570 2746 50  0000 L CNN
+F 1 "10k" H 7570 2655 50  0000 L CNN
+F 2 "Resistor_SMD:R_0805_2012Metric" V 7430 2700 50  0001 C CNN
+F 3 "~" H 7500 2700 50  0001 C CNN
+	1    7500 2700
+	1    0    0    -1
+$EndComp
+Wire Wire Line
+	7500 2550 7500 2500
+$Comp
+L power:GND #PWR0143
+U 1 1 5DCD8890
+P 7500 2900
+F 0 "#PWR0143" H 7500 2650 50  0001 C CNN
+F 1 "GND" H 7505 2727 50  0000 C CNN
+F 2 "" H 7500 2900 50  0001 C CNN
+F 3 "" H 7500 2900 50  0001 C CNN
+	1    7500 2900
+	1    0    0    -1
+$EndComp
+Wire Wire Line
+	7500 2900 7500 2850
+Wire Wire Line
+	7750 2150 7750 2500
+Wire Wire Line
+	7750 2500 7500 2500
+Connection ~ 7500 2500
+Wire Wire Line
+	7500 2500 7500 2450
 $EndSCHEMATC
